Commit message: Revise URDF

File: Prototype_URDF/kumo.urdf (robot description, URDF)
Before this commit: robot kumo, 9 links, 8 joints
Joints:
- removed joint Rev4-1
- added joint Rev1-4: type continuous, parent base_link, child leg_link1-4, origin xyz=-0.0332 0.021 0.0358 rpy=0 0 -0.7853, axis 0.0 0.0 -1.0
- joint Rev1-1: origin xyz=0.0332 -0.021 0.0358 rpy=0 0 0 -> xyz=0.0332 -0.021 0.0358 rpy=0 0 -0.7853
- joint Rev1-2: origin xyz=0.0332 0.021 0.0358 rpy=0 0 0 -> xyz=0.0332 0.021 0.0358 rpy=0 0 0.7853
- joint Rev1-3: origin xyz=-0.0332 -0.021 0.0358 rpy=0 0 0 -> xyz=-0.0332 -0.021 0.0358 rpy=0 0 0.7853
- joint Rev2-1: axis -0.707107 -0.707107 0.0 -> -0.0 -1.0 0.0; origin xyz=-0.000707 -0.02291 -0.0123 rpy=0 0 0 -> xyz=0.0157 -0.0167 -0.0123 rpy=0 0 0
- joint Rev2-2: axis 0.707107 -0.707107 0.0 -> -0.0 -1.0 0.0; origin xyz=-0.000707 -0.06491 -0.0123 rpy=0 0 0 -> xyz=0.0157 -0.0587 -0.0123 rpy=0 0 0
- joint Rev2-3: axis -0.707107 0.707107 0.0 -> 0.0 1.0 0.0; origin xyz=0.065693 -0.02291 -0.0123 rpy=0 0 0 -> xyz=-0.0157 0.0167 -0.0123 rpy=0 0 0
- joint Rev4-2: axis 0.707107 0.707107 0.0 -> 0.0 1.0 0.0; origin xyz=0.065693 -0.06491 -0.0123 rpy=0 0 0 -> xyz=-0.0157 0.0167 -0.0123 rpy=0 0 0
